Commit message: Velodyne model rotated 180º on X axis

File: robots_description/models/iris_velodyne/model.xacro (robot description, xacro)
@@ -15,5 +15,5 @@
   <xacro:include filename="$(find velodyne_description)/urdf/HDL-32E.urdf.xacro"/>
   <HDL-32E parent="base_link" name="velodyne" topic="/velodyne_points" hz="10" samples="220" gpu="true">
-    <origin xyz="0 0 0" rpy="0 0 0" />
+    <origin xyz="0 0 0" rpy="3.14 0 0" />
   </HDL-32E>
   <!-- macros for gazebo plugins, sensors -->
